Commit message: horrible ccommit but it muse be made.
Signed-off-by: Joas329 <joaquinphilco@hotmail.com>

File: description/robotic_arm_2.urdf (robot description, URDF)
Before this commit: robot RoboticArmv2, 7 links, 6 joints
Links:
- removed link Link1
- added link Link7, mass 0.0135263682638669; collision mesh filename=package://arm_control/description/meshes/Link7.STL; visual mesh filename=package://arm_control/description/meshes/Link7.STL
- link Link2: mass 0.577415758791343 -> 0.970074967448887
- link Link3: mass 0.251663957012598 -> 0.577415758791343
- link Link4: mass 0.356013835274962 -> 0.251663957012598
- link Link5: mass 0.175482504091363 -> 0.300029723918034
- link Link6: mass 0.0135263682638669 -> 0.155889261418066
- link base_link: mass 4.037 -> 0.83438
Joints:
- removed joint J1
- added joint J7: type revolute, parent Link6, child Link7, origin xyz=0.02775 0 -0.001 rpy=0 0 0, axis 1 0 0, limit lower=0 upper=6.28 effort=0 velocity=0
- joint J2: axis 0 0 -1 -> 0 1 0; limit lower=-1.57 upper=1.57 effort=0 velocity=0 -> lower=0 upper=6.2832 effort=10 velocity=10; origin xyz=0 0.134 0 rpy=0 0 0 -> xyz=0 0 0 rpy=1.5708 0 0; parent Link1 -> base_link
- joint J3: axis 0 0 -1 -> 0 0 1; limit lower=0 upper=3.14 effort=10 velocity=10 -> lower=-1.5708 upper=1.5708 effort=10 velocity=10; origin xyz=0 0.322 0 rpy=0 0 0 -> xyz=0 0.14 0 rpy=0 0 0
- joint J4: axis 1 0 0 -> 0 0 1; limit lower=-3.14 upper=3.14 effort=10 velocity=10 -> lower=0 upper=6.28 effort=10 velocity=10; origin xyz=0.03 0 0 rpy=0 0 0 -> xyz=0 0.322 0 rpy=0 0 0
- joint J5: axis 0 0 -1 -> 1 0 0; limit lower=-1.57 upper=1.57 effort=10 velocity=10 -> lower=0 upper=6.28 effort=10 velocity=10; origin xyz=0.20275 0 0 rpy=3.1416 0 0 -> xyz=0.03 0 0 rpy=0 0 0
- joint J6: axis 1 0 0 -> 0 0 1; limit lower=-3.14 upper=3.14 effort=10 velocity=10 -> lower=0 upper=6.28 effort=0 velocity=0; origin xyz=0.02825 0 -0.01 rpy=-3.1416 0 0 -> xyz=0.20275 0 0 rpy=0 0 0

File: description/robotic_arm_3.urdf (robot description, URDF)
Before this commit: robot RoboticArmv2, 7 links, 6 joints
Links:
- removed link Link1
- added link Link7, mass 0.0135263682638669; collision mesh filename=package://arm_control/description/meshes/Link7.STL; visual mesh filename=package://arm_control/description/meshes/Link7.STL
- link Link2: mass 0.577415758791343 -> 0.97007
- link Link3: mass 0.251663957012598 -> 0.577415758791342
- link Link4: mass 0.356013835274962 -> 0.251663957012598
- link Link5: mass 0.175482504091363 -> 0.300029724080392
- link Link6: mass 0.0135263682638669 -> 0.155889261418066
- link base_link: mass 4.037 -> 0.83438
Joints:
- joint J1: axis 0 -1 0 -> 0 1 0; child Link1 -> Link2; limit lower=-3.14 upper=3.14 effort=10 velocity=10 -> lower=0 upper=6.28 effort=10 velocity=10; origin xyz=0 0 0.0059964 rpy=1.5708 0 0 -> xyz=0 0 0 rpy=1.5708 0 0
- joint J2: axis 0 0 -1 -> 0 0 1; child Link2 -> Link3; limit lower=-1.57 upper=1.57 effort=0 velocity=0 -> lower=-1.570796 upper=1.570796 effort=10 velocity=10; origin xyz=0 0.134 0 rpy=0 0 0 -> xyz=0 0.14 0 rpy=0 0 0; parent Link1 -> Link2
- joint J3: axis 0 0 -1 -> 0 0 1; child Link3 -> Link4; limit lower=0 upper=3.14 effort=10 velocity=10 -> lower=-1.5708 upper=1.5708 effort=10 velocity=10; parent Link2 -> Link3
- joint J4: child Link4 -> Link5; limit lower=-3.14 upper=3.14 effort=10 velocity=10 -> lower=0 upper=6.28 effort=10 velocity=10; parent Link3 -> Link4
- joint J5: axis 0 0 -1 -> 0 0 1; child Link5 -> Link6; limit lower=-1.57 upper=1.57 effort=10 velocity=10 -> lower=-1.570796 upper=1.570796 effort=10 velocity=10; parent Link4 -> Link5
- joint J6: child Link6 -> Link7; limit lower=-3.14 upper=3.14 effort=10 velocity=10 -> lower=0 upper=6.28 effort=10 velocity=10; parent Link5 -> Link6
