Commit message: yurs/description: Add placeholder joint limits.
Signed-off-by: Joas329 <joaquinphilco@hotmail.com>

File: description/yurs_base_station.urdf.xacro (robot description, xacro)
@@ -1,3 +1,3 @@
-<?xml version="1.0" encoding="utf-8"?>
+<?xml version="1.0"?>
 <!-- This URDF was automatically created by SolidWorks to URDF Exporter! Originally created by Stephen Brawner (brawner@gmail.com)
      Commit Version: 1.6.0-4-g7f85cfe  Build Version: 1.6.7995.38578
@@ -70,5 +70,5 @@
     <child link="$(arg namespace)_link1" />
     <axis xyz="0 -1 0" />
-    <limit lower="0" upper="0" effort="0" velocity="0" />
+    <limit lower="-1.57" upper="1.57" effort="1000" velocity="1.0" />
   </joint>
   <!-- ################# Link 2 ################# -->
@@ -106,5 +106,5 @@
     <child link="$(arg namespace)_link2" />
     <axis xyz="0 0 1" />
-    <limit lower="0" upper="0" effort="0" velocity="0" />
+    <limit lower="-1.57" upper="1.57" effort="1000" velocity="1.0" />
   </joint>
   <!-- ################# Link 3 ################# -->
@@ -142,5 +142,5 @@
     <child link="$(arg namespace)_link3" />
     <axis xyz="0 0 1" />
-    <limit lower="0" upper="0" effort="0" velocity="0" />
+    <limit lower="-1.57" upper="1.57" effort="1000" velocity="1.0" />
   </joint>
   <!-- ################# Link 4 ################# -->
@@ -178,5 +178,5 @@
     <child link="$(arg namespace)_link4" />
     <axis xyz="1 0 0" />
-    <limit lower="0" upper="0" effort="0" velocity="0" />
+    <limit lower="-1.57" upper="1.57" effort="1000" velocity="1.0" />
   </joint>
   <!-- ################# Link 5 ################# -->
@@ -214,5 +214,5 @@
     <child link="$(arg namespace)_link5" />
     <axis xyz="0 0 1" />
-    <limit lower="0" upper="0" effort="0" velocity="0" />
+    <limit lower="-1.57" upper="1.57" effort="1000" velocity="1.0" />
   </joint>
   <!-- ################# Link 6 ################# -->
@@ -250,5 +250,5 @@
     <child link="$(arg namespace)_link6" />
     <axis xyz="-1 0 0" />
-    <limit lower="0" upper="0" effort="0" velocity="0" />
+    <limit lower="-1.57" upper="1.57" effort="1000" velocity="1.0" />
   </joint>
 </robot>

Commit message: yurs/description: Add real joint limits to robot description.
Signed-off-by: Joas329 <joaquinphilco@hotmail.com>

File: description/yurs_base_station.urdf.xacro (robot description, xacro)
@@ -70,5 +70,5 @@
     <child link="$(arg namespace)_link1" />
     <axis xyz="0 -1 0" />
-    <limit lower="-1.57" upper="1.57" effort="1000" velocity="1.0" />
+    <limit lower="-0.785398" upper="0.785398" effort="1000" velocity="1.0" />
   </joint>
   <!-- ################# Link 2 ################# -->
@@ -106,5 +106,5 @@
     <child link="$(arg namespace)_link2" />
     <axis xyz="0 0 1" />
-    <limit lower="-1.57" upper="1.57" effort="1000" velocity="1.0" />
+    <limit lower="-1.5708" upper="0.7854" effort="1000" velocity="1.0" />
   </joint>
   <!-- ################# Link 3 ################# -->
@@ -142,5 +142,5 @@
     <child link="$(arg namespace)_link3" />
     <axis xyz="0 0 1" />
-    <limit lower="-1.57" upper="1.57" effort="1000" velocity="1.0" />
+    <limit lower="0.174533" upper="4.53786" effort="1000" velocity="1.0" />
   </joint>
   <!-- ################# Link 4 ################# -->
@@ -178,5 +178,5 @@
     <child link="$(arg namespace)_link4" />
     <axis xyz="1 0 0" />
-    <limit lower="-1.57" upper="1.57" effort="1000" velocity="1.0" />
+    <limit lower="-3.1416" upper="3.1416" effort="1000" velocity="1.0" />
   </joint>
   <!-- ################# Link 5 ################# -->
@@ -214,5 +214,5 @@
     <child link="$(arg namespace)_link5" />
     <axis xyz="0 0 1" />
-    <limit lower="-1.57" upper="1.57" effort="1000" velocity="1.0" />
+    <limit lower="-1.5708" upper="1.5708" effort="1000" velocity="1.0" />
   </joint>
   <!-- ################# Link 6 ################# -->
@@ -250,5 +250,5 @@
     <child link="$(arg namespace)_link6" />
     <axis xyz="-1 0 0" />
-    <limit lower="-1.57" upper="1.57" effort="1000" velocity="1.0" />
+    <limit lower="-1.5708" upper="1.5708" effort="1000" velocity="1.0" />
   </joint>
 </robot>
