Commit message: desccription/macros: Add a default value (robot1) for namespace parameter.
Signed-off-by: Joas329 <joaquinphilco@hotmail.com>

File: description/macros.xacro (robot description, xacro)
@@ -85,5 +85,5 @@
         <origin xyz="${x*intom} ${-z*intom} ${y*intom}" rpy="${roll} ${pitch} ${yaw}"/>
     </xacro:macro>
-    <xacro:macro name="arm_component" params="namespace component_number type parent_link child_link mass axis Lxx Lxy Lxz Lyy Lyz Lzz file inertiaX inertiaY inertiaZ effort_limit lower_limit upper_limit velocity_limit joint_X joint_Y joint_Z">
+    <xacro:macro name="arm_component" params="component_number type parent_link child_link mass axis Lxx Lxy Lxz Lyy Lyz Lzz file inertiaX inertiaY inertiaZ effort_limit lower_limit upper_limit velocity_limit joint_X joint_Y joint_Z namespace:='robot1'">
         <link name="${namespace}_arm_a${component_number}">
             <visual>
