Commit message: description: Use robot1 namespace prefix in the ROS2 controller macro.
Signed-off-by: Joas329 <joaquinphilco@hotmail.com>

File: description/arm.ros2_control.xacro (robot description, xacro)
@@ -1,6 +1,6 @@
 <?xml version="1.0"?>
 <robot xmlns:xacro="http://www.ros.org/wiki/xacro">
-  <xacro:macro name="ar_ros2_control" params="
-    ar_model
+  <xacro:macro name="arm_ros2_control" params="
+    arm_model
     plugin_name
     serial_port
@@ -17,8 +17,8 @@
     <xacro:property name="driver_parameters"
       value="${xacro.load_yaml(driver_parameters_file)}"/>
-    <ros2_control name="${ar_model}" type="system">
+    <ros2_control name="${arm_model}" type="system">
       <hardware>
         <plugin>${plugin_name}</plugin>
-        <param name="ar_model">${ar_model}</param>
+        <param name="arm_model">${arm_model}</param>
         <param name="serial_port">${serial_port}</param>
         <param name="calibrate">${calibrate}</param>
@@ -27,5 +27,6 @@
         <param name="tf_prefix">${tf_prefix}</param>
       </hardware>
-      <joint name="${tf_prefix}joint_1">
+      <xacro:property name="ns" value="${tf_prefix}"/>
+      <joint name="${ns}arm_j1">
         <command_interface name="position">
           <param name="min">${robot_parameters['j1_limit_min']}</param>
@@ -41,5 +42,5 @@
         <param name="position_offset">${joint_offset_parameters['joint_1']}</param>
       </joint>
-      <joint name="${tf_prefix}joint_2">
+      <joint name="${ns}arm_j2">
         <command_interface name="position">
           <param name="min">${robot_parameters['j2_limit_min']}</param>
@@ -55,5 +56,5 @@
         <param name="position_offset">${joint_offset_parameters['joint_2']}</param>
       </joint>
-      <joint name="${tf_prefix}joint_3">
+      <joint name="${ns}arm_j3">
         <command_interface name="position">
           <param name="min">${robot_parameters['j3_limit_min']}</param>
@@ -69,5 +70,5 @@
         <param name="position_offset">${joint_offset_parameters['joint_3']}</param>
       </joint>
-      <joint name="${tf_prefix}joint_4">
+      <joint name="${ns}arm_j4">
         <command_interface name="position">
           <param name="min">${robot_parameters['j4_limit_min']}</param>
@@ -83,5 +84,5 @@
         <param name="position_offset">${joint_offset_parameters['joint_4']}</param>
       </joint>
-      <joint name="${tf_prefix}joint_5">
+      <joint name="${ns}arm_j5">
         <command_interface name="position">
           <param name="min">${robot_parameters['j5_limit_min']}</param>
@@ -97,5 +98,5 @@
         <param name="position_offset">${joint_offset_parameters['joint_5']}</param>
       </joint>
-      <joint name="${tf_prefix}joint_6">
+      <joint name="${ns}arm_j6">
         <command_interface name="position">
           <param name="min">${robot_parameters['j6_limit_min']}</param>
